File: hardware/telesoarer.sch (KiCad schematic (older format))
At the start: 52 parts, among them IC1 STM32F103CBT6, K1 RC_SIG, P1 PZ, P2 PZ_IN, P3 OLED 0.91\" 128x32, P4 AOUT, P5 CONN_01X05, Q1 BC847C, U1 MS5611, U2 MCP1703T-3302, U3 AD8027ARTZ, X1 16MHz

Commit message: PCB progress check-in
Parts:
- BOOT0: renamed from R2; footprint footprints:R_0603 -> footprints:BR_O_0603
Connections:
- net SWDCLK: now also P5.4 (P4); no longer P5.2 (P2)
- net SWDIO: now also P5.5 (P5); no longer P5.3 (P3)
- net USART1_RX: now also P5.3 (P3); no longer P5.5 (P5)
- net USART1_TX: now also P5.2 (P2); no longer P5.4 (P4)
Changed lines of the file:
@@
 Wire Wire Line
 	1250 3050 1500 3050
-Text Label 1500 2950 0    60   ~ 0
+Text Label 1500 3150 0    60   ~ 0
 USART1_RX
-Text Label 1500 3050 0    60   ~ 0
+Text Label 1500 3250 0    60   ~ 0
 USART1_TX
 Wire Wire Line
@@
 20 E0 57 DC FC 57 73 5D 07 14 FC 3B B8 FE 8A E6 FF 5B AF AF 5C AC AF 9F 81 6F 5A FD 7F 8D 89 FD
 CB D3 8E 5B 2D BF 2A 35 7F 55 A3 B5 A5 5D 7D 4C 00 C0 FF 07 AF 49 E4 EC 18 E0 49 D6 00 00 00 00
-49 45 4E 44 AE 42 60 82 00
+49 45 4E 44 AE 42 60 82 C8
 EndData
 $EndBitmap
@@
 SWDCLK
 $Comp
-L R R2
+L R BOOT0
 U 1 1 5822A331
 P 3050 6000
-F 0 "R2" V 3130 6000 50  0000 C CNN
+F 0 "BOOT0" V 3130 6000 50  0000 C CNN
 F 1 "NC" V 3050 6000 50  0000 C CNN
-F 2 "footprints:R_0603" H 3050 6000 60  0001 C CNN
+F 2 "footprints:BR_O_0603" H 3050 6000 60  0001 C CNN
 F 3 "" H 3050 6000 60  0001 C CNN
 	1    3050 6000
@@
 Wire Wire Line
 	1250 3250 1500 3250
-Text Label 1500 3150 0    60   ~ 0
+Text Label 1500 2950 0    60   ~ 0
 SWDIO
-Text Label 1500 3250 0    60   ~ 0
+Text Label 1500 3050 0    60   ~ 0
 SWDCLK
 $Comp
