File: hardware/telesoarer.sch (KiCad schematic (older format))
At the start: 52 parts, among them IC1 STM32F103CBT6, J1 BOOT0, J2 RESET, K1 RC_SIG, P1 PZ, P2 PZ_IN, P3 OLED 0.91\" 128x32, P4 AOUT, P5 CONN_01X05, Q1 BC847C, U1 MS5611, U2 MCP1703T-3302, U3 AD8027ARTZ, X1 16MHz

Commit message: MILESTONE: PCB Routing Completed (FINAL DRAFT 1)
Parts:
- P4: footprint footprints:PIN_ARRAY_2X1 -> Pin_Headers:Pin_Header_Angled_1x02
Changed lines of the file:
@@
 F 0 "P4" H 10600 5250 50  0000 C CNN
 F 1 "AOUT" H 10800 5100 50  0000 C CNN
-F 2 "footprints:PIN_ARRAY_2X1" H 10600 5100 50  0001 C CNN
+F 2 "Pin_Headers:Pin_Header_Angled_1x02" H 10600 5100 50  0001 C CNN
 F 3 "" H 10600 5100 50  0000 C CNN
 	1    10600 5100
