File: hardware/telesoarer.kicad_pcb (KiCad board)
At the start: 2 copper layers, 72.8 x 16.5 mm, 52 parts, among them IC1 STM32F103CBT6, K1 RC_SIG, P1 PZ, P2 PZ_IN, P3 OLED 0.91" 128x32, P4 AOUT, P5 CONN_01X05, Q1 BC847C, U1 MS5611, U2 MCP1703T-3302, U3 AD8027ARTZ, X1 16MHz

Commit message: PCB progress check-in
Parts:
- removed R2: NC, footprints:R_0603
- added BOOT0: NC, footprints:BR_O_0603, F.Cu at (38.4, 28.3)
- added BOOT0: NC, footprints:BR_O_0603, F.Cu at (69.1, 57.5)
- moved R11 47.7 mm to (52.8, 51.2), turned to 180 degrees
- moved C13 46.2 mm to (43.8, 51.8)
- moved R10 45.5 mm to (52.8, 49.7), turned to 180 degrees
- moved R8 45.0 mm to (50.5, 51.2)
- moved C11 43.3 mm to (41.1, 55.9)
- moved R7 43.1 mm to (50.5, 49.7)
- moved C12 42.9 mm to (43.8, 49.8)
- moved R9 40.6 mm to (48.1, 28.2), turned to 270 degrees
- moved C1 40.3 mm to (41.0, 26.9), turned to 270 degrees
- moved D5 38.7 mm to (41.3, 60.1)
- moved C14 36.4 mm to (43.8, 53.1)
- moved Q1 35.8 mm to (50.4, 28.6)
- moved C18 34.2 mm to (51.7, 33.3), turned to 180 degrees
- moved R14 34.2 mm to (55.0, 51.1)
- moved P2 33.7 mm to (61.6, 28.1)
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Connections:
- IC1 pad 10: (no net) -> Net-(IC1-Pad10)
- IC1 pad 11: (no net) -> Net-(IC1-Pad11)
- IC1 pad 12: (no net) -> Net-(IC1-Pad12)
- IC1 pad 2: (no net) -> Net-(IC1-Pad2)
- IC1 pad 21: (no net) -> Net-(IC1-Pad21)
- IC1 pad 22: (no net) -> Net-(IC1-Pad22)
- IC1 pad 29: (no net) -> Net-(IC1-Pad29)
- IC1 pad 3: (no net) -> Net-(IC1-Pad3)
- IC1 pad 38: (no net) -> Net-(IC1-Pad38)
- IC1 pad 39: (no net) -> Net-(IC1-Pad39)
- IC1 pad 4: (no net) -> Net-(IC1-Pad4)
- IC1 pad 40: (no net) -> Net-(IC1-Pad40)
- IC1 pad 41: (no net) -> Net-(IC1-Pad41)
- IC1 pad 42: (no net) -> Net-(IC1-Pad42)
- IC1 pad 45: (no net) -> Net-(IC1-Pad45)
- IC1 pad 46: (no net) -> Net-(IC1-Pad46)
- P5 pad 2: /SWDCLK -> /USART1_TX
- P5 pad 3: /SWDIO -> /USART1_RX
- P5 pad 4: /USART1_TX -> /SWDCLK
- P5 pad 5: /USART1_RX -> /SWDIO
- U3 pad 5: (no net) -> Net-(U3-Pad5)
Routing:
- net +BATT: track 25.0 -> 74.9 mm, vias 2 -> 4
- net GND: track 19.9 -> 44.9 mm, vias 0 -> 6
- net Net-(IC1-Pad13): track 0.00 -> 22.0 mm, vias 0 -> 2
- net /SCK: track 0.00 -> 17.2 mm, vias 0 -> 2
- net /MISO: track 0.00 -> 16.3 mm, vias 0 -> 2
- net /MOSI: track 0.00 -> 15.5 mm, vias 0 -> 2
- net Net-(L1-Pad1): track 19.5 -> 34.6 mm, vias 0 -> 2
- net /VARIO_~SS: track 0.00 -> 14.2 mm, vias 0 -> 2
- net +3V3: track 2.45 -> 9.89 mm, vias 0 -> 1
- net Net-(BOOT0-Pad1): track 0.00 -> 6.04 mm
- net Net-(Q1-Pad1): track 0.00 -> 1.29 mm
- added copper zone on In1.Cu, net +3V3
- added copper zone on In2.Cu, net GND
Other:
- board size 72.8 x 16.5 mm -> 87.4 x 22 mm
- copper layers 2 -> 4
- net class +3V3 added: clearance 0.1524, trace_width 0.508, via_dia 1.524, via_drill 0.508
- net class +5V removed
- net class Default: via_dia 0.6858 -> 0.889
- net class GND: via_dia 0.8636 -> 1.524; via_drill 0.4572 -> 0.508

Commit message: PCB work continues
Parts:
- removed BOOT0 (x2): NC, footprints:BR_O_0603
- removed R7: NC, footprints:R_0402
- added J1: BOOT0, footprints:BR_O_0603, F.Cu at (39.1, 28.4)
- added J2: RESET, footprints:BR_O_0603, F.Cu at (39.1, 26.8)
- moved P4 52.1 mm to (28.6, 43.2)
- moved R15 27.5 mm to (31.9, 42.6), turned to 90 degrees
- moved R8 27.1 mm to (37.0, 27.7), turned to 0 degrees
- moved R12 22.0 mm to (33.1, 42.8), turned to 90 degrees
- moved D4 18.6 mm to (47.9, 46.0)
- moved D5 18.6 mm to (48.1, 42.8)
- moved R13 17.9 mm to (38.4, 42.9), turned to 90 degrees
- moved R14 16.8 mm to (50.6, 34.9), turned to 90 degrees
- moved C10 16.0 mm to (36.5, 39.2), turned to 180 degrees
- moved R11 15.7 mm to (39.5, 42.9), turned to 270 degrees
- moved C16 15.7 mm to (50.4, 41.7)
- moved C15 15.5 mm to (50.3, 40.4)
- moved C14 12.9 mm to (35.1, 43.6)
- moved C11 12.7 mm to (40.8, 43.2), turned to 90 degrees
- moved R10 12.6 mm to (41.9, 43.3), turned to 90 degrees
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Routing:
- net /USART1_TX: track 0.00 -> 28.4 mm, vias 0 -> 2
- net /LED_BLUE: track 0.00 -> 23.3 mm, vias 0 -> 2
- net GND: track 44.9 -> 67.6 mm, vias 6 -> 11
- net /SWDIO: track 0.00 -> 22.2 mm, vias 0 -> 2
- net /LED_RED: track 0.00 -> 21.2 mm, vias 0 -> 2
- net Net-(IC1-Pad43): track 0.00 -> 20.1 mm, vias 0 -> 3
- net /~RESET: track 0.00 -> 16.2 mm, vias 0 -> 2
- net /LED_GREEN: track 0.00 -> 14.4 mm, vias 0 -> 2
- net +3V3: track 9.89 -> 21.6 mm, vias 1 -> 7
- net Net-(P4-Pad2): track 0.00 -> 11.4 mm, vias 0 -> 1
- net Net-(R13-Pad2): track 0.00 -> 11.3 mm, vias 0 -> 2
- net Net-(C14-Pad1): track 0.00 -> 6.88 mm
- net Net-(C11-Pad1): track 0.00 -> 2.71 mm
- net /SIG: track 0.00 -> 2.48 mm
- net +BATT: track 74.9 -> 77.4 mm
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