File: hardware/telesoarer.kicad_pcb (KiCad board)
At the start: 4 copper layers, 87.4 x 22 mm, 52 parts, among them IC1 STM32F103CBT6, J1 BOOT0, J2 RESET, K1 RC_SIG, P1 PZ, P2 PZ_IN, P3 OLED 0.91" 128x32, P4 AOUT, P5 CONN_01X05, Q1 BC847C, U1 MS5611, U2 MCP1703T-3302, U3 AD8027ARTZ, X1 16MHz

Commit message: More PCB work
Parts:
- moved D4 10.6 mm to (49.7, 35.6)
- moved D5 8.54 mm to (49.7, 34.4)
- moved R14 2.56 mm to (51.9, 32.6)
- moved C17 1.15 mm to (50.5, 31.8)
- moved C18 1.10 mm to (52.1, 31.2)
Routing:
- net /OVBAT2: track 0.00 -> 2.13 mm
- net +3V3: track 21.6 -> 23.6 mm, vias 7 -> 8
- net /OVBAT1: track 0.00 -> 1.86 mm
- net /VBAT: track 0.00 -> 1.14 mm
Changed lines of the file:
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@@
   (general
     (links 120)
-    (no_connects 31)
+    (no_connects 27)
     (area 25.349199 25.349199 112.803201 47.456401)
     (thickness 1.6)
     (drawings 26)
-    (tracks 419)
+    (tracks 428)
     (zones 0)
     (modules 52)
@@
   )
   (module footprints:R_0402 (layer F.Cu)
-    (at 50.6095 34.8615 90)
+    (at 51.8795 32.639 90)
     (descr "Resistor SMD 0402, reflow soldering, Vishay (see dcrcw.pdf)")
     (tags "resistor 0402")
@@
   )
   (module footprints:C_0402 (layer F.Cu)
-    (at 50.419 32.893 90)
+    (at 50.546 31.75 90)
     (descr "Capacitor SMD 0402, reflow soldering, AVX (see smccp.pdf)")
     (tags "capacitor 0402")
@@
   )
   (module footprints:C_0402 (layer F.Cu)
-    (at 51.943 32.3215 180)
+    (at 52.1335 31.242 180)
     (descr "Capacitor SMD 0402, reflow soldering, AVX (see smccp.pdf)")
     (tags "capacitor 0402")
@@
       (rotate (xyz 0 0 0))
     )
-  )
-  (module Diodes_SMD:SOD-523 (layer F.Cu)
-    (at 47.9425 45.974)
-    (descr "http://www.diodes.com/datasheets/ap02001.pdf p.144")
-    (tags "Diode SOD523")
-    (attr smd)
-    (fp_text reference D4 (at 0 -1.5) (layer F.SilkS)
-      (effects (font (size 1 1) (thickness 0.15)))
-    )
-    (fp_text value D_Schottky (at 4.318 0) (layer F.Fab)
-      (effects (font (size 0.508 0.508) (thickness 0.127)))
-    )
-    (fp_line (start -0.4 0.6) (end 1.15 0.6) (layer F.SilkS) (width 0.15))
-    (fp_line (start -0.4 -0.6) (end 1.15 -0.6) (layer F.SilkS) (width 0.15))
-    (pad 2 smd rect (at -0.7 0) (size 0.6 0.7) (layers F.Cu F.Paste F.Mask)
-      (net 31 /OVBAT1))
-    (pad 1 smd rect (at 0.7 0) (size 0.6 0.7) (layers F.Cu F.Paste F.Mask)
-      (net 28 /VBAT))
-  )
-  (module Diodes_SMD:SOD-523 (layer F.Cu)
-    (at 48.0695 42.799)
-    (descr "http://www.diodes.com/datasheets/ap02001.pdf p.144")
-    (tags "Diode SOD523")
-    (attr smd)
-    (fp_text reference D5 (at 0 -1.5) (layer F.SilkS)
-      (effects (font (size 1 1) (thickness 0.15)))
-    )
-    (fp_text value D_Schottky (at 3.937 0.127) (layer F.Fab)
-      (effects (font (size 0.508 0.508) (thickness 0.127)))
-    )
-    (fp_line (start -0.4 0.6) (end 1.15 0.6) (layer F.SilkS) (width 0.15))
-    (fp_line (start -0.4 -0.6) (end 1.15 -0.6) (layer F.SilkS) (width 0.15))
-    (pad 2 smd rect (at -0.7 0) (size 0.6 0.7) (layers F.Cu F.Paste F.Mask)
-      (net 32 /OVBAT2))
-    (pad 1 smd rect (at 0.7 0) (size 0.6 0.7) (layers F.Cu F.Paste F.Mask)
-      (net 28 /VBAT))
   )
   (module Pin_Headers:Pin_Header_Angled_1x03 (layer F.Cu)
@@
       (rotate (xyz 0 0 0))
     )
+  )
+  (module Diodes_SMD:SOD-523 (layer F.Cu)
+    (at 49.7205 34.417)
+    (descr "http://www.diodes.com/datasheets/ap02001.pdf p.144")
+    (tags "Diode SOD523")
+    (attr smd)
+    (fp_text reference D5 (at -0.508 -2.413) (layer F.SilkS)
+      (effects (font (size 0.508 0.508) (thickness 0.127)))
+    )
+    (fp_text value D_Schottky (at -15.748 3.6195) (layer F.Fab) hide
+      (effects (font (size 1 1) (thickness 0.15)))
+    )
+    (fp_line (start -0.4 0.6) (end 1.15 0.6) (layer F.SilkS) (width 0.15))
+    (fp_line (start -0.4 -0.6) (end 1.15 -0.6) (layer F.SilkS) (width 0.15))
+    (pad 2 smd rect (at -0.7 0) (size 0.6 0.7) (layers F.Cu F.Paste F.Mask)
+      (net 32 /OVBAT2))
+    (pad 1 smd rect (at 0.7 0) (size 0.6 0.7) (layers F.Cu F.Paste F.Mask)
+      (net 28 /VBAT))
+  )
+  (module Diodes_SMD:SOD-523 (layer F.Cu)
+    (at 49.7205 35.56)
+    (descr "http://www.diodes.com/datasheets/ap02001.pdf p.144")
+    (tags "Diode SOD523")
+    (attr smd)
+    (fp_text reference D4 (at -0.127 -2.3495) (layer F.SilkS)
+      (effects (font (size 0.508 0.508) (thickness 0.127)))
+    )
+    (fp_text value D_Schottky (at -15.748 1.27) (layer F.Fab) hide
+      (effects (font (size 1 1) (thickness 0.15)))
+    )
+    (fp_line (start -0.4 0.6) (end 1.15 0.6) (layer F.SilkS) (width 0.15))
+    (fp_line (start -0.4 -0.6) (end 1.15 -0.6) (layer F.SilkS) (width 0.15))
+    (pad 2 smd rect (at -0.7 0) (size 0.6 0.7) (layers F.Cu F.Paste F.Mask)
+      (net 31 /OVBAT1))
+    (pad 1 smd rect (at 0.7 0) (size 0.6 0.7) (layers F.Cu F.Paste F.Mask)
+      (net 28 /VBAT))
   )
   (gr_line (start 58.42 44.45) (end 58.42 25.4) (angle 90) (layer Edge.Cuts) (width 0.1016))
@@
   (segment (start 40.4964 31.0984) (end 39.3192 31.0984) (width 0.3048) (layer F.Cu) (net 5))
   (segment (start 40.6252 31.2272) (end 40.4964 31.0984) (width 0.3048) (layer F.Cu) (net 5))
-  (segment (start 48.387 32.893) (end 48.387 32.131) (width 0.3048) (layer F.Cu) (net 5))
-  (segment (start 48.0716 34.2244) (end 48.387 33.909) (width 0.3048) (layer F.Cu) (net 5))
-  (segment (start 48.387 33.909) (end 48.387 32.893) (width 0.3048) (layer F.Cu) (net 5))
-  (via (at 48.387 32.893) (size 0.889) (drill 0.3302) (layers F.Cu B.Cu) (net 5))
   (segment (start 47.2252 34.2244) (end 48.0716 34.2244) (width 0.3048) (layer F.Cu) (net 5))
   (segment (start 48.091 31.835) (end 47.498 31.835) (width 0.3048) (layer F.Cu) (net 5))
@@
   (segment (start 35.2132 37.1164) (end 34.9882 36.8914) (width 0.1524) (layer F.Cu) (net 5))
   (segment (start 39.3192 31.0984) (end 38.3032 31.0984) (width 0.254) (layer F.Cu) (net 5))
+  (segment (start 48.387 32.893) (end 48.387 32.131) (width 0.3048) (layer F.Cu) (net 5))
+  (segment (start 48.387 33.909) (end 48.387 32.893) (width 0.3048) (layer F.Cu) (net 5))
+  (via (at 48.387 32.893) (size 0.889) (drill 0.3302) (layers F.Cu B.Cu) (net 5))
+  (segment (start 48.0716 34.2244) (end 48.387 33.909) (width 0.3048) (layer F.Cu) (net 5))
   (segment (start 51.435 28.575) (end 51.435 27.559) (width 0.508) (layer F.Cu) (net 6))
   (segment (start 61.857 27.567) (end 63.5325 27.567) (width 0.508) (layer F.Cu) (net 6))
@@
   (via (at 33.3375 40.3225) (size 0.889) (drill 0.3302) (layers F.Cu B.Cu) (net 14))
   (segment (start 35.3695 42.3545) (end 43.561 42.3545) (width 0.1524) (layer B.Cu) (net 14))
+  (segment (start 47.2252 33.7244) (end 45.4084 33.7244) (width 0.1524) (layer F.Cu) (net 15) (status 400000))
+  (via (at 45.2755 33.5915) (size 0.889) (drill 0.3302) (layers F.Cu B.Cu) (net 15))
+  (segment (start 45.4084 33.7244) (end 45.2755 33.5915) (width 0.1524) (layer F.Cu) (net 15))
   (segment (start 36.5705 27.686) (end 36.5705 29.406) (width 0.1524) (layer F.Cu) (net 15))
   (segment (start 37.5285 28.448) (end 36.5125 29.464) (width 0.2286) (layer F.Cu) (net 15))
@@
   (segment (start 40.767 43.73) (end 41.883 43.73) (width 0.1524) (layer F.Cu) (net 24))
   (segment (start 41.883 43.73) (end 41.91 43.757) (width 0.1524) (layer F.Cu) (net 24))
+  (segment (start 50.4205 35.56) (end 50.4205 34.417) (width 0.1524) (layer F.Cu) (net 28) (status C00000))
+  (segment (start 47.2252 35.7244) (end 48.8561 35.7244) (width 0.1524) (layer F.Cu) (net 31) (status C00000))
+  (segment (start 48.8561 35.7244) (end 49.0205 35.56) (width 0.1524) (layer F.Cu) (net 31) (status C00000))
+  (segment (start 47.2252 35.2244) (end 47.8971 35.2244) (width 0.1524) (layer F.Cu) (net 32) (status 400000))
+  (segment (start 48.7045 34.417) (end 49.0205 34.417) (width 0.1524) (layer F.Cu) (net 32) (status 800000))
+  (segment (start 47.8971 35.2244) (end 48.7045 34.417) (width 0.1524) (layer F.Cu) (net 32))
   (segment (start 40.8305 39.497) (end 40.5765 39.497) (width 0.1524) (layer F.Cu) (net 34))
   (segment (start 40.1252 39.9483) (end 40.1252 40.8244) (width 0.1524) (layer F.Cu) (net 34))

Commit message: If I don't quit now, I may find myself divorced. To the morrow, then!
Routing:
- net /USART1_RX: track 0.00 -> 28.1 mm, vias 0 -> 2
- net /SWDCLK: track 0.00 -> 21.0 mm, vias 0 -> 3
- net /SWDIO: track 22.2 -> 23.1 mm
- net Net-(IC1-Pad13): track 22.2 -> 22.9 mm

Commit message: MILESTONE: PCB Routing Completed (FINAL DRAFT 1)
Parts:
- P4: footprint footprints:PIN_ARRAY_2X1 -> Pin_Headers:Pin_Header_Angled_1x02
- moved PZ1 42.7 mm to (71.9, 27.4), turned to 180 degrees
- moved L1 36.4 mm to (69.1, 35.7)
- moved R1 6.73 mm to (26.9, 29.0)
- moved U2 3.74 mm to (29.8, 33.5), turned to 90 degrees
- moved P5 3.74 mm to (32.0, 28.4), turned to 180 degrees
- moved K1 3.67 mm to (26.9, 36.6)
- moved C5 3.64 mm to (32.4, 33.6), turned to 270 degrees
- moved C16 3.47 mm to (50.1, 38.2), turned to 180 degrees
- moved C13 3.05 mm to (50.1, 40.7), turned to 270 degrees
- moved R15 2.62 mm to (29.3, 42.3)
- moved R14 1.85 mm to (50.1, 33.1), turned to 180 degrees
- moved P4 1.74 mm to (26.9, 42.9), turned to 180 degrees
- moved C15 1.25 mm to (50.1, 39.2)
- moved C4 1.24 mm to (29.3, 37.9)
- moved D1 1.09 mm to (31.6, 35.9)
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Routing:
- net GND: track 67.6 -> 152.8 mm, vias 11 -> 24
- net /OLED_~SS: track 0.00 -> 21.7 mm, vias 0 -> 2
- net /OLED_D/~C: track 0.00 -> 19.9 mm, vias 0 -> 2
- net /OLED_~RES: track 0.00 -> 15.3 mm, vias 0 -> 2
- net /SCK: track 16.1 -> 27.9 mm, vias 2 -> 3
- net Net-(L1-Pad1): track 34.6 -> 25.5 mm
- net +3V3: track 23.8 -> 32.7 mm
- net /MOSI: track 15.6 -> 22.9 mm, vias 2 -> 3
- net /VBAT: track 1.14 -> 7.35 mm
- net /LED_BLUE: track 23.3 -> 18.7 mm
- net Net-(C17-Pad1): track 0.00 -> 3.86 mm
- net (no net): track 3.69 -> 0.00 mm
- net Net-(P3-Pad13): track 0.00 -> 3.62 mm
- net /USART1_RX: track 28.1 -> 25.0 mm
- net Net-(C12-Pad1): track 0.00 -> 2.94 mm
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- added copper zone on F.Cu, net GND
- added copper zone on In1.Cu, net GND
- removed copper zone on B.Cu, net +BATT
- removed copper zone on F.Cu, net +BATT
Other:
- board size 87.4 x 22 mm -> 50.3 x 19.1 mm
- net class Default: via_dia 0.889 -> 0.762
- board text added: "github.com/gruvin/telesoarer"
- board text removed: "github.com/ gruvin/telesoarer"
