File: hardware/_saved_telesoarer.sch (KiCad schematic (older format))
At the start: 52 parts, among them IC1 STM32F103CBT6, K1 RC_SIG, P1 PZ, P2 PZ_IN, P3 OLED 0.91\" 128x32, P4 AOUT, P5 CONN_01X05, Q1 BC847C, U1 MS5611, U2 MCP1703T-3302, U3 AD8027ARTZ, X1 16MHz

Commit message: PCB work continues
Parts:
- gave numbers to parts that had none: 2
Changed lines of the file:
@@
 20 E0 57 DC FC 57 73 5D 07 14 FC 3B B8 FE 8A E6 FF 5B AF AF 5C AC AF 9F 81 6F 5A FD 7F 8D 89 FD
 CB D3 8E 5B 2D BF 2A 35 7F 55 A3 B5 A5 5D 7D 4C 00 C0 FF 07 AF 49 E4 EC 18 E0 49 D6 00 00 00 00
-49 45 4E 44 AE 42 60 82 C8
+49 45 4E 44 AE 42 60 82 00
 EndData
 $EndBitmap
@@
 SWDCLK
 $Comp
-L R J?
+L R J1
 U 1 1 5822A331
 P 3050 6000
-F 0 "J?" V 2950 6000 50  0000 C CNN
+F 0 "J1" V 2950 6000 50  0000 C CNN
 F 1 "BOOT0" V 3150 6000 50  0000 C CNN
 F 2 "footprints:BR_O_0603" H 3050 6000 60  0001 C CNN
@@
 	6100 5550 6200 5550
 $Comp
-L R J?
+L R J2
 U 1 1 5836AF4F
 P 5700 5800
-F 0 "J?" H 5600 5750 50  0000 C CNN
+F 0 "J2" H 5600 5750 50  0000 C CNN
 F 1 "RESET" H 5550 5850 50  0000 C CNN
 F 2 "footprints:BR_O_0603" V 5630 5800 50  0001 C CNN

Commit message: sub module won't sync
Parts:
- D4, D5: footprint Diodes_SMD:SOD-523 -> Diodes_SMD:SOD-323
Changed lines of the file:
@@
 F 0 "D4" H 7450 2550 50  0000 C CNN
 F 1 "D_Schottky" H 7450 2350 50  0001 C CNN
-F 2 "Diodes_SMD:SOD-523" H 7450 2450 50  0001 C CNN
+F 2 "Diodes_SMD:SOD-323" H 7450 2450 50  0001 C CNN
 F 3 "" H 7450 2450 50  0000 C CNN
 	1    7450 2450
@@
 F 0 "D5" H 7450 2850 50  0000 C CNN
 F 1 "D_Schottky" H 7450 2950 50  0001 C CNN
-F 2 "Diodes_SMD:SOD-523" H 7450 2750 50  0001 C CNN
+F 2 "Diodes_SMD:SOD-323" H 7450 2750 50  0001 C CNN
 F 3 "" H 7450 2750 50  0000 C CNN
 	1    7450 2750
